Commit message: feature: robot bisualization on simulation

File: rave_description/urdf/rave.urdf.xacro (robot description, xacro)
@@ -28,6 +28,6 @@
       <plugin name="gazebo_ros_controller_manager" filename="libgazebo_ros_control.so">
           <legacyModeNS>true</legacyModeNS>
-          <robotNamespace>${robot_namespace}</robotNamespace>
-          <!-- <robotSimType>steer_bot_hardware_gazebo/SteerBotHardwareGazebo</robotSimType--> -->
+          <!-- <robotNamespace>${robot_namespace}</robotNamespace> -->
+          <robotSimType>steer_bot_hardware_gazebo/SteerBotHardwareGazebo</robotSimType>
       </plugin>
   </gazebo>

File: rave_description/urdf/wheel.urdf.xacro (robot description, xacro)
@@ -13,5 +13,5 @@
 		<link name="${wheel_prefix}_steer_link">
 			<visual>
-				<origin xyz="0 0 0" rpy="0 0 0"/>
+				<origin xyz="0 0 0" rpy="0 0 1.0"/>
 				<geometry>
 					<cylinder radius="${steer_radius}" length="${steer_thickness}"/>
@@ -37,8 +37,8 @@
 			</inertial>
 			<visual>
-				<origin xyz="0 0 0" rpy="0 0 0" />
+				<origin xyz="0 0 0" rpy="${M_PI/2} 0 0" />
 				<geometry>
-					<mesh filename="package://rave_description/meshes/wheel.stl" />
-					<!-- <cylinder length="${wheel_length}" radius="${wheel_radius}" /> -->
+					<!-- <mesh filename="package://rave_description/meshes/wheel.stl" /> -->
+					<cylinder length="${wheel_length}" radius="${wheel_radius}" />
 				</geometry>
 				<material name="black" />
@@ -107,8 +107,8 @@
 			</inertial>
 			<visual>
-				<origin xyz="0 0 0" rpy="0 0 0" />
+				<origin xyz="0 0 0" rpy="${M_PI/2} 0 0" />
 				<geometry>
-					<mesh filename="package://rave_description/meshes/wheel.stl" />
-					<!-- <cylinder length="${wheel_length}" radius="${wheel_radius}" /> -->
+					<!-- <mesh filename="package://rave_description/meshes/wheel.stl" /> -->
+					<cylinder length="${wheel_length}" radius="${wheel_radius}" />
 				</geometry>
 				<material name="black" />

Commit message: wrong controller

File: rave_description/urdf/rave.urdf.xacro (robot description, xacro)
@@ -14,14 +14,4 @@
   <xacro:property name="wheel_length" value="0.1143" />
   <xacro:property name="wheel_radius" value="0.1651" />
-  <!-- Gazebo plugins -->
-  <!-- Load ros_control plugin using the steer_bot_hardware_gazebo
-  implementation of the hardware_interface::RobotHW -->
-  <!-- <gazebo>
-    <plugin name="gazebo_ros_control" filename="libgazebo_ros_control.so">
-      <robotNamespace>${robot_namespace}</robotNamespace>
-      <robotSimType>steer_bot_hardware_gazebo/SteerBotHardwareGazebo</robotSimType>
-      <legacyModeNS>false</legacyModeNS>
-    </plugin>
-  </gazebo> -->
   <gazebo>
       <!--ROS Control Plugin -->
@@ -89,7 +79,7 @@
     <link name="base_footprint"/>
     <joint name="base_footprint_joint" type="fixed">
-    <parent link="base_link" />
-    <child link="base_footprint" />
-    <origin xyz="0 0 -${wheel_radius}" rpy="0 0 0" />
+      <parent link="base_link" />
+      <child link="base_footprint" />
+      <origin xyz="0 0 -${wheel_radius}" rpy="0 0 0" />
     </joint>
   <!-- Rave wheel macros -->
